Commit message: fix urdf frames and remove of unnecesary folder

File: lexium_digital_twin/urdf/Lexium_Cobot_L03S_3D-simpl.SLDASM.urdf (robot description, URDF)
Before this commit: robot Lexium_Cobot_L03S_3D-simpl.SLDASM, 7 links, 6 joints
Links:
- link Link_1: mass 0.88431 -> 0.884295316293331
- link Link_2: mass 2.3218 -> 2.32175993259425
- link Link_3: mass 1.2033 -> 1.20330042207005
- link Link_4: mass 0.4932 -> 0.493200863231089
- link Link_5: mass 0.55157 -> 0.55156964581296
- link Link_6: mass 0.095133 -> 0.0951327910810692
- link base_link: mass 0.46037 -> 0.460374564690923
Joints:
- joint Joint_1: limit lower=-3.14159 upper=3.14159 effort=100 velocity=2.0 -> lower=0 upper=0 effort=0 velocity=0; origin xyz=0 0 0.08605 rpy=0 0 0 -> xyz=0 0 0.08605 rpy=0 0 -3.14159
- joint Joint_2: axis 0 0 1 -> 0 0 -1; limit lower=-3.14159 upper=3.14159 effort=100 velocity=2.0 -> lower=0 upper=0 effort=0 velocity=0; origin xyz=0.016544 0.047713 0.0645 rpy=1.5708 0 2.8078 -> xyz=0 -0.0505 0.0644999999999995 rpy=-1.5707963267949 1.5707963267949 3.14159265358979
- joint Joint_3: axis 0 0 -1 -> 0 0 1; limit lower=-3.14159 upper=3.14159 effort=100 velocity=2.0 -> lower=0 upper=0 effort=0 velocity=0; origin xyz=0.23513 -0.072328 -0.0035 rpy=3.1416 0 3.1416 -> xyz=0 -0.24600000094683 -0.00350000000001006 rpy=-3.14159265358979 0 -3.14159265358979
- joint Joint_4: limit lower=-3.14159 upper=3.14159 effort=100 velocity=2.0 -> lower=0 upper=0 effort=0 velocity=0; origin xyz=-0.11206 0.19856 -0.0245 rpy=-3.1416 0 0 -> xyz=0 -0.228000000001584 -0.0244999999969376 rpy=-3.14159265356148 0 -1.5707963267949
- joint Joint_5: axis 0 0 -1 -> 0 0 1; limit lower=-3.14159 upper=3.14159 effort=100 velocity=2.0 -> lower=0 upper=0 effort=0 velocity=0; origin xyz=-0.018336 -0.073755 0.0415 rpy=-1.5708 0.34315 2.8979 -> xyz=0 0.0760000000011137 0.0414999999977316 rpy=1.57079632682321 0 -3.14159265358979
- joint Joint_6: axis 0 0 -1 -> 0 0 1; limit lower=-3.14159 upper=3.14159 effort=100 velocity=2.0 -> lower=0 upper=0 effort=0 velocity=0; origin xyz=-0.059775 -0.046936 0.0415 rpy=-1.5708 0.36234 2.2365 -> xyz=0 -0.0760000000025846 0.0414999999985123 rpy=-1.5707963267949 0.785398163 -3.14159265358979
