Commit message: Added moveitconfig pkg. Lexium trajectory server (lexium_moveit). Modbus pos commander (lexium_digital_twin).

File: src/lexium_digital_twin/urdf/Lexium_Cobot_L03S_3D-simpl.SLDASM.urdf (robot description, URDF)
Before this commit: robot lexium_digital_twin, 7 links, 6 joints
Joints:
- joint Joint_1: limit lower=0 upper=0 effort=0 velocity=0 -> lower=0 upper=360 effort=0 velocity=0
- joint Joint_2: limit lower=0 upper=0 effort=0 velocity=0 -> lower=0 upper=360 effort=0 velocity=0
- joint Joint_3: limit lower=0 upper=0 effort=0 velocity=0 -> lower=0 upper=360 effort=0 velocity=0
- joint Joint_4: limit lower=0 upper=0 effort=0 velocity=0 -> lower=0 upper=360 effort=0 velocity=0
- joint Joint_5: limit lower=0 upper=0 effort=0 velocity=0 -> lower=0 upper=360 effort=0 velocity=0
- joint Joint_6: limit lower=0 upper=0 effort=0 velocity=0 -> lower=0 upper=360 effort=0 velocity=0

Commit message: Unfinished version of moveit. Corrected position ofssets. Now visualizes phantom and allows for point arriving (unoptimized path planning). Added bridge to send trajectory server and bridge node to send pos.

File: src/lexium_digital_twin/urdf/Lexium_Cobot_L03S_3D-simpl.SLDASM.urdf (robot description, URDF)
Before this commit: robot lexium_digital_twin, 7 links, 6 joints
Joints:
- joint Joint_1: limit lower=0 upper=360 effort=0 velocity=0 -> lower=-6.2831 upper=6.2831 effort=150 velocity=2
- joint Joint_2: limit lower=0 upper=360 effort=0 velocity=0 -> lower=-6.2831 upper=6.2831 effort=150 velocity=2
- joint Joint_3: limit lower=0 upper=360 effort=0 velocity=0 -> lower=-6.2831 upper=6.2831 effort=150 velocity=2
- joint Joint_4: limit lower=0 upper=360 effort=0 velocity=0 -> lower=-6.2831 upper=6.2831 effort=150 velocity=2
- joint Joint_5: limit lower=0 upper=360 effort=0 velocity=0 -> lower=-6.2831 upper=6.2831 effort=150 velocity=2
- joint Joint_6: limit lower=0 upper=360 effort=0 velocity=0 -> lower=-6.2831 upper=6.2831 effort=150 velocity=2

Commit message: Added workcell with piston and slider. Upgraded visuals and added sliders to joint testing without hardware

File: src/lexium_digital_twin/urdf/Lexium_Cobot_L03S_3D-simpl.SLDASM.urdf (robot description, URDF)
Before this commit: robot lexium_digital_twin, 7 links, 6 joints
Joints:
- joint Joint_1: limit lower=0 upper=0 effort=0 velocity=0 -> lower=-3.14159 upper=3.14159 effort=150.0 velocity=3.15
- joint Joint_2: limit lower=0 upper=0 effort=0 velocity=0 -> lower=-3.14159 upper=3.14159 effort=150.0 velocity=3.15
- joint Joint_3: limit lower=0 upper=0 effort=0 velocity=0 -> lower=-3.14159 upper=3.14159 effort=150.0 velocity=3.15
- joint Joint_4: limit lower=0 upper=0 effort=0 velocity=0 -> lower=-3.14159 upper=3.14159 effort=28.0 velocity=3.2
- joint Joint_5: limit lower=0 upper=0 effort=0 velocity=0 -> lower=-3.14159 upper=3.14159 effort=28.0 velocity=3.2
- joint Joint_6: limit lower=0 upper=0 effort=0 velocity=0 -> lower=-3.14159 upper=3.14159 effort=28.0 velocity=3.2
