Commit message: Added basic routine for workstation

File: src/lexium_digital_twin/urdf/workcell.urdf.xacro (robot description, xacro)
@@ -108,5 +108,5 @@
     </collision>
   </link>
-  <joint name="rail_joint" type="prismatic">
+  <joint name="rail_joint" type="fixed">
     <parent link="workcell_base"/>
     <child link="rail_link"/>
@@ -146,5 +146,5 @@
     </collision>
   </link>
-  <joint name="piston_joint" type="prismatic">
+  <joint name="piston_joint" type="fixed">
     <parent link="workcell_base"/>
     <child link="piston_link"/>
@@ -157,5 +157,5 @@
     <parent link="workcell_base"/>
     <child link="base_link"/>
-    <origin xyz="0.0 0.0 0.0" rpy="0 0 0"/>
+    <origin xyz="0.0 0.0 0.0" rpy="0 0 135"/>
   </joint>
 </robot>
